File: pcb/control_board_2/control_board_2.kicad_pcb (KiCad board)
At the start: 2 copper layers, 85 x 55 mm, 8 parts, among them J1 JST4 VH Power, SW2 Mode Switch

Commit message: He was forced to pay $40 PCB shipping AGAIN
Other:
- board text added: "Overblinking Control Board V2 4/17/2026"
- board text removed: "Overblinking Control Board V2 4/13/2026"
Changed lines of the file:
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@@
 			(drillshape 0)
 			(scaleselection 1)
-			(outputdirectory "C:/Users/pluh/Documents/2026Spring/EECE598/pcb/control_board_1/gerbers/")
+			(outputdirectory "gerbers/")
 		)
 	)
@@
 		)
 	)
-	(gr_text "Overblinking\nControl Board V2\n4/13/2026"
+	(gr_text "Overblinking\nControl Board V2\n4/17/2026"
 		(at 89 60 30)
 		(layer "B.SilkS")
